File: pcb/ArduinoNano LearningBot 3-30-18.sch (EAGLE design)
At the start: 13 parts

Commit message: footprints confirmed
Parts:
- removed BATTERYPACK: (no value), SparkFun-Connectors:M02PTH
- removed LDR1, LDR2: (no value), SparkFun-Connectors:M02LOCK
- removed LDR_RESISTOR1, LDR_RESISTOR2: 10k, SparkFun-Passives:RESISTORPTH-1/4W
- removed SWITCH: 332-12, con-garry:332-12
- added J1: (no value), SparkFun-Connectors:CONN_03-SCREW-5MM
- added LED1, LED2, LED3, LED4, LED5, LED6: WS2812B5050, adafruit:WS2812B5050
- added R2: (no value), pot:3RP/1610N-VERTICAL
- added S2: (no value), switch-omron:10-XX
- added S3: (no value), ArduinoNano LearningBot 3-15-18:SWITCH_320-938
- added SP1: SPEAKER/AL60P, adafruit:SPEAKER/AL60P
- U$1: value NANO -> ARDUINO-CLONE_NANO; device Arduino-clone:NANO -> ArduinoNano LearningBot 3-15-18:ARDUINO-CLONE_NANO
Connections:
- removed net GND: BATTERYPACK.1, SWITCH-1.S
- removed net GNDARDUINO: SWITCH-5.S, U$1.GND2
- removed net RAW: BATTERYPACK.2, SWITCH-2.S
- net A0: now also U$1.D8; no longer LDR2.2, LDR_RESISTOR1.1, U$1.A1
- net A1: now also U$1.D9; no longer LDR1.2, LDR_RESISTOR2.1, U$1.A0
- net ARDUINORAW: now also U$1.TX0; no longer SWITCH-6.S, U$1.RAW
- net GND-ISO: now also U$1.RX1; no longer LDR_RESISTOR1.2, LDR_RESISTOR2.2, U$1.GND
- net IRLED: now also U$1.A7; no longer U$1.D2
- net IRRECEIVER: now also U$1.A5; no longer U$1.D4
- net SERVO1: now also U$1.A4; no longer U$1.D5
- net SERVO2: now also U$1.A6; no longer U$1.D3
- net ULTRASONICSENSOR: now also U$1.A2; no longer U$1.D7
- net VCC: now also U$1.GND2; no longer LDR1.1, LDR2.1, U$1.5.5V
Other:
- moved on the sheet: ULTRASONICSENSOR
