File: pcb/ArduinoNano LearningBot 4-2-18.brd (EAGLE design)
At the start: 106.9 x 60.1 mm, 21 parts

Commit message: yes
Parts:
- removed LED1, LED2, LED3, LED4, LED5, LED6: WS2812B5050, adafruit:WS2812B
- added LED-1, LED-2, LED-3, LED-4, LED-5, LED-6: WS2812B5050, adafruit:WS2812B
- moved SERVO2 18.0 mm to (44.7, 7.77), turned to 90 degrees
- moved SERVO1 17.4 mm to (71.4, 7.77), turned to 90 degrees
- moved BATTERY_CONNECTOR 7.43 mm to (76.2, 19.7), turned to 45 degrees
- moved ULTRASONICSENSOR 2.01 mm to (54.4, 48.6)
- moved LDR1 1.91 mm to (88.9, 59.1)
- moved LDR2 1.91 mm to (17.8, 59.1)
- moved U$1 0.63 mm to (55.5, 34.5)
Connections:
- removed net DIGITAL_PUSHBUTTON_PIN: DIGITAL_PUSHBUTTON.1, U$1.D4
- removed net N$5: LED4.2-DOUT, LED6.4-DIN
- removed net N$7: POTENTIOMETER.3, U$1.A4
- new net BUTTON: DIGITAL_PUSHBUTTON.1, U$1.D8
- new net LED-1: LED-1.4-DIN, U$1.D6
- new net N$9: BATTERY_CONNECTOR.1, POWER_SWITCH.NO1
- new net POTPIN: POTENTIOMETER.2, U$1.A4
- new net RAWIN: BATTERY_CONNECTOR.2, U$1.RAW
- net GND: now also LED-1.3-GND, LED-2.3-GND, LED-3.3-GND, LED-4.3-GND, LED-5.3-GND, LED-6.3-GND, POTENTIOMETER.1, POWER_SWITCH.NC1; no longer LED1.3-GND, LED2.3-GND, LED3.3-GND, LED4.3-GND, LED5.3-GND, LED6.3-GND, POTENTIOMETER.2
- net IR_SENSOR1_AO: now also U$1.A1; no longer U$1.A3
- net IR_SENSOR2_AO: now also U$1.A2; no longer POWER_SWITCH.NC1, U$1.A1
- net IR_SENSOR2_DO: now also U$1.D5; no longer U$1.D9
- net LDR1_AO: now also U$1.A0; no longer U$1.A2
- net LDR2_AO: now also U$1.A3; no longer U$1.A0
- net LDR2_DO: now also U$1.D4; no longer U$1.D8
- net N$1: now also LED-3.2-DOUT, LED-4.4-DIN; no longer LED2.4-DIN, U$1.D10
- net N$2: now also LED-4.2-DOUT, LED-5.4-DIN; no longer LED1.4-DIN, LED2.2-DOUT
- net N$4: now also LED-5.2-DOUT, LED-6.4-DIN; no longer LED1.2-DOUT, LED4.4-DIN
- net N$6: now also LED-1.2-DOUT, LED-2.4-DIN; no longer LED3.4-DIN, LED6.2-DOUT
- net N$8: now also LED-2.2-DOUT, LED-3.4-DIN; no longer LED3.2-DOUT, LED5.4-DIN
- net SERVO1_PIN: now also U$1.D11; no longer U$1.D6
- net SERVO2_PIN: now also U$1.D10; no longer U$1.D5
- net TOUCH_SENSOR: now also U$1.D9; no longer U$1.D2
- net VCC: now also LED-1.1-VDD, LED-2.1-VDD, LED-3.1-VDD, LED-4.1-VDD, LED-5.1-VDD, LED-6.1-VDD, POTENTIOMETER.3, U$1.5V; no longer LED1.1-VDD, LED2.1-VDD, LED3.1-VDD, LED4.1-VDD, LED5.1-VDD, LED6.1-VDD, POTENTIOMETER.1
Routing:
- net N$1: track 0.00 -> 151.4 mm, vias 0 -> 4
- net VCC: track 0.00 -> 97.8 mm, vias 0 -> 3
- net LDR1_DO: track 0.00 -> 82.3 mm
- net LDR1_AO: track 0.00 -> 73.2 mm, vias 0 -> 2
- net GND: track 0.00 -> 67.5 mm, vias 0 -> 6
- net LDR2_AO: track 0.00 -> 62.8 mm, vias 0 -> 1
- net LDR2_DO: track 0.00 -> 62.7 mm
- net IR_SENSOR1_DO: track 0.00 -> 58.6 mm
- net IR_SENSOR2_AO: track 0.00 -> 48.1 mm, vias 0 -> 2
- net SPEAKERPIN: track 0.00 -> 46.6 mm
- net POTPIN: track 0.00 -> 40.4 mm, vias 0 -> 1
- net ULTRASONICSENSOR_PIN: track 0.00 -> 39.2 mm
- net IR_SENSOR1_AO: track 0.00 -> 39.0 mm, vias 0 -> 2
- net IR_SENSOR2_DO: track 0.00 -> 37.7 mm
- net SERVO1_PIN: track 0.00 -> 35.8 mm
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- added copper zone on layer 16, net GND
- added copper zone on layer 1, net VCC
Other:
- board size 106.9 x 60.1 mm -> 106.9 x 61.4 mm
