File: pcb/LearningBot v0.2/ArduinoNano LearningBot 4-23-18.brd (EAGLE design)
At the start: 106.9 x 58.9 mm, 21 parts

Commit message: Hi
Parts:
- moved U$1 5.83 mm to (51.8, 29.5)
- moved DIGITAL_PUSHBUTTON 5.00 mm to (30.2, 39.0)
- moved IRSENSOR1 5.00 mm to (68.9, 43.8)
- moved IRSENSOR2 5.00 mm to (48.5, 43.8)
- moved LED-1 5.00 mm to (31.0, 52.2)
- moved LED-2 5.00 mm to (7.35, 28.6)
- moved LED-3 5.00 mm to (7.35, 52.2)
- moved LED-4 5.00 mm to (77.0, 52.2)
- moved LED-5 5.00 mm to (101.4, 52.2)
- moved LED-6 5.00 mm to (101.4, 28.6)
- moved POTENTIOMETER 5.00 mm to (100.8, 40.5)
- moved POWER_SWITCH 5.00 mm to (72.9, 18.2)
- moved PUSHBUTTON_RESISTOR 5.00 mm to (18.0, 27.1)
- moved SERVO1 5.00 mm to (68.4, 3.77)
- moved SERVO2 5.00 mm to (39.8, 3.77)
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Other:
- board size 106.9 x 58.9 mm -> 106.9 x 60.9 mm
- board text added: "LearningBot V0.2"
