File: pcb/v0.2/ArduinoNano LearningBot 4-21-18.sch (EAGLE design)
At the start: 19 parts

Commit message: almost there!
Connections:
- removed net GND-ISO: LED1.GND, LED2.GND, LED3.GND, LED4.GND, R2.2, SENSOR1.2, SENSOR2.2, SENSOR3.2, SENSOR4.2, SERVO1.1, SERVO2.1, SPEAKER.+, U$1.GND2, ULTRA.4, VR1.A
- removed net N.C.: S11.S, U$1.GND
- new net GND: LED1.GND, LED2.GND, LED3.GND, LED4.GND, R2.2, S11.S, SENSOR1.2, SENSOR2.2, SENSOR3.2, SENSOR4.2, SERVO1.1, SERVO2.1, SPEAKER.+, U$1.GND, U$1.GND2, ULTRA.4, VR1.A
Changed lines of the file:
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@@
 <?xml version="1.0" encoding="utf-8"?>
 <!DOCTYPE eagle SYSTEM "eagle.dtd">
-<eagle version="8.4.0">
+<eagle version="8.4.1">
 <drawing>
 <settings>
@@
 </segment>
 </net>
-<net name="N.C." class="0">
-<segment>
-<wire x1="121.92" y1="66.04" x2="116.84" y2="66.04" width="0.1524" layer="91"/>
-<pinref part="S1" gate="1" pin="S"/>
-<label x="119.38" y="66.04" size="1.778" layer="95"/>
-</segment>
-<segment>
-<pinref part="GND20" gate="G$1" pin="GND-ISO"/>
-<pinref part="U$1" gate="G$1" pin="GND"/>
-<wire x1="139.7" y1="104.14" x2="144.78" y2="104.14" width="0.1524" layer="91"/>
-<wire x1="144.78" y1="104.14" x2="144.78" y2="81.28" width="0.1524" layer="91"/>
-</segment>
-</net>
 <net name="SERVO2_PIN" class="0">
 <segment>
@@
 </segment>
 </net>
-<net name="GND-ISO" class="0">
+<net name="GND" class="0">
 <segment>
 <pinref part="VR1" gate="G$1" pin="A"/>
@@
 <pinref part="GND15" gate="G$1" pin="GND-ISO"/>
 </segment>
-</net>
+<segment>
+<wire x1="121.92" y1="66.04" x2="116.84" y2="66.04" width="0.1524" layer="91"/>
+<pinref part="S1" gate="1" pin="S"/>
+<label x="119.38" y="66.04" size="1.778" layer="95"/>
+</segment>
+<segment>
+<pinref part="GND20" gate="G$1" pin="GND-ISO"/>
+<pinref part="U$1" gate="G$1" pin="GND"/>
+<wire x1="139.7" y1="104.14" x2="144.78" y2="104.14" width="0.1524" layer="91"/>
+<wire x1="144.78" y1="104.14" x2="144.78" y2="81.28" width="0.1524" layer="91"/>
+</segment>
+</net>
