File: pcb/v0.2/ArduinoNano LearningBot 4-21-18.sch (EAGLE design)
At the start: 19 parts

Commit message: component placement 95%
Parts:
- removed DIGITAL_PUSHBUTTON: (no value), switch-omron:10-XX
- removed IRSENSOR1, LDR1: (no value), SparkFun-Connectors:M04LOCK
- removed POTENTIOMETER: (no value), pot:3RP/1610N-VERTICAL
- removed PUSHBUTTON_RESISTOR: 10k, SparkFun-Passives:RESISTORPTH-1/4W
- removed TOUCH_SENSOR_RESISTOR: 10MOhm, SparkFun-Passives:RESISTORPTH-1/4W
- added BUTTON: (no value), switch-omron:10-XX
- added R1: 10MOhm, SparkFun-Passives:RESISTORPTH-1/4W
- added R2: 10k, SparkFun-Passives:RESISTORPTH-1/4W
- added SENSOR1, SENSOR2: (no value), SparkFun-Connectors:M04LOCK
- added VR1: (no value), pot:3RP/1610N-VERTICAL
- renumbered BATTERY_CONNECTOR to BAT, IRSENSOR2 to SENSOR3, LDR2 to SENSOR4, LED-2 to LED1, LED-3 to LED2, LED-5 to LED3, LED-6 to LED4, ULTRASONICSENSOR to ULTRA
Connections:
- net IR_SENSOR2_AO renamed SENSOR3
- net LDR2_AO renamed SENSOR4
- removed net CAP_TOUCH_SEND_PIN: TOUCH_SENSOR_RESISTOR.2, U$1.A5
- removed net GND: IRSENSOR1.2, LDR1.2, LED1.GND, LED2.GND, LED3.GND, LED4.GND, POTENTIOMETER.A, PUSHBUTTON_RESISTOR.2, S11.S, SENSOR3.2, SENSOR4.2, SERVO1.1, SERVO2.1, SPEAKER.+, U$1.GND, U$1.GND2, ULTRA.4
- removed net IR_SENSOR1_AO: IRSENSOR1.4, U$1.A1
- removed net LDR1_AO: LDR1.4, U$1.A0
- removed net SERVOVCC: SERVO1.2, SERVO2.2
- new net GND-ISO: LED1.GND, LED2.GND, LED3.GND, LED4.GND, R2.2, SENSOR1.2, SENSOR2.2, SENSOR3.2, SENSOR4.2, SERVO1.1, SERVO2.1, SPEAKER.+, U$1.GND2, ULTRA.4, VR1.A
- new net LEDS: U$1.D9
- new net N$6: SERVO1.3, U$1.D11
- new net N.C.: S11.S, U$1.GND
- new net SENSOR1: SENSOR1.4, U$1.A0
- new net SENSOR2: SENSOR2.4, U$1.A1
- new net TOUCH: R1.2, U$1.A5
- net BUTTON: now also BUTTON.S; no longer DIGITAL_PUSHBUTTON.S
- net CAP_TOUCH_RECEIVE_PIN: now also R1.1; no longer TOUCH_SENSOR_RESISTOR.1
- net IR_SENSOR1_DO: now also SENSOR2.3; no longer IRSENSOR1.3
- net LDR1_DO: now also SENSOR1.3; no longer LDR1.3
- net LED-1: no longer U$1.D9
- net N$3: now also BUTTON.S1, R2.1; no longer DIGITAL_PUSHBUTTON.S1, PUSHBUTTON_RESISTOR.1
- net POTPIN: now also VR1.E; no longer POTENTIOMETER.E
- net VCC: now also BUTTON.P, BUTTON.P1, SENSOR1.1, SENSOR2.1, SERVO1.2, SERVO2.2, VR1.S; no longer DIGITAL_PUSHBUTTON.P1, IRSENSOR1.1, LDR1.1, POTENTIOMETER.S, SERVO1.3, U$1.D11
Other:
- moved on the sheet: SERVO1, SERVO2, SPEAKER

Commit message: changes to physical
Parts:
- BAT: value (none) -> BAT
- S1: value (none) -> POWER
Changed lines of the file:
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@@
 <part name="SUPPLY17" library="SparkFun-Aesthetics" deviceset="VCC" device=""/>
 <part name="SUPPLY4" library="SparkFun-Aesthetics" deviceset="VCC" device=""/>
-<part name="BAT" library="SparkFun-Connectors" deviceset="M03" device="POLAR"/>
+<part name="BAT" library="SparkFun-Connectors" deviceset="M03" device="POLAR" value="BAT"/>
 <part name="R1" library="SparkFun-Passives" deviceset="RESISTOR" device="PTH-1/4W" value="10MOhm"/>
-<part name="S1" library="ArduinoNano LearningBot 4-21-18" deviceset="SWITCH_320-938" device=""/>
+<part name="S1" library="ArduinoNano LearningBot 4-21-18" deviceset="SWITCH_320-938" device="" value="POWER"/>
 <part name="GND11" library="SparkFun-Aesthetics" deviceset="GND-ISO" device=""/>
 <part name="GND9" library="SparkFun-Aesthetics" deviceset="GND-ISO" device=""/>
