File: pcb/v0.2/ArduinoNano LearningBot 4-21-18.sch (EAGLE design)
At the start: 19 parts

Commit message: Howdy
Parts:
- added U$2: TOUCHSENSOR, CapTouch:TOUCHSENSOR
Connections:
- removed net LED-1: LED1.DI
- net LEDS: now also LED1.DI
- net TOUCH: now also U$2.1
Changed lines of the file:
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@@
 <part name="GND14" library="SparkFun-Aesthetics" deviceset="GND-ISO" device=""/>
 <part name="GND15" library="SparkFun-Aesthetics" deviceset="GND-ISO" device=""/>
+<part name="U$2" library="CapTouch" deviceset="TOUCHSENSOR" device=""/>
 </parts>
 <sheets>
@@
 <attribute name="VALUE" x="104.14" y="96.52" size="1.778" layer="96" display="off"/>
 </instance>
+<instance part="U$2" gate="G$2" x="205.74" y="63.5"/>
 </instances>
 <busses>
@@
 </segment>
 </net>
-<net name="LED-1" class="0">
-<segment>
-<pinref part="LED1" gate="G$1" pin="DI"/>
-<wire x1="175.26" y1="198.12" x2="200.66" y2="198.12" width="0.1524" layer="91"/>
-<label x="175.26" y="198.12" size="1.778" layer="95"/>
-</segment>
-</net>
 <net name="N$9" class="0">
 <segment>
@@
 <wire x1="162.56" y1="116.84" x2="162.56" y2="63.5" width="0.1524" layer="91"/>
 <pinref part="R1" gate="G$1" pin="2"/>
-<label x="203.2" y="63.5" size="1.778" layer="95"/>
 <wire x1="162.56" y1="63.5" x2="203.2" y2="63.5" width="0.1524" layer="91"/>
+<pinref part="U$2" gate="G$2" pin="1"/>
 </segment>
 </net>
@@
 <label x="68.58" y="129.54" size="1.778" layer="95"/>
 </segment>
-</net>
+<segment>
+<pinref part="LED1" gate="G$1" pin="DI"/>
+<wire x1="175.26" y1="198.12" x2="200.66" y2="198.12" width="0.1524" layer="91"/>
+<label x="175.26" y="198.12" size="1.778" layer="95"/>
+</segment>
+</net>
