File: pcb/v0.2/ArduinoNano LearningBot 4-21-18.brd (EAGLE design)
At the start: 106.9 x 58.9 mm, 19 parts

Commit message: New Board
Parts:
- BATTERY_CONNECTOR: device SparkFun-Connectors:JST-3-PTH-VERT -> SparkFun-Connectors:MOLEX-1X3
- moved SPEAKER 28.5 mm to (36.0, 24.0)
- moved LED-5 26.9 mm to (79.0, 47.5)
- moved LED-2 25.6 mm to (6.00, 25.0)
- moved LED-3 19.2 mm to (27.5, 47.5)
- moved LED-6 17.9 mm to (100.0, 25.0)
- moved DIGITAL_PUSHBUTTON 14.4 mm to (22.0, 34.0)
- moved S1 13.0 mm to (72.0, 15.0)
- moved IRSENSOR2 11.1 mm to (41.0, 44.0)
- moved LDR1 10.1 mm to (93.0, 44.0)
- moved PUSHBUTTON_RESISTOR 9.94 mm to (17.0, 22.0)
- moved LDR2 9.81 mm to (21.0, 44.0)
- moved TOUCH_SENSOR_RESISTOR 8.94 mm to (65.8, 27.6)
- moved POTENTIOMETER 7.81 mm to (76.8, 34.5), turned to 225 degrees
- moved BATTERY_CONNECTOR 7.81 mm to (28.4, 14.6), turned to 313.5 degrees
- moved SERVO1 6.64 mm to (67.0, 2.77)
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Other:
- board size 106.9 x 58.9 mm -> 106.9 x 55.1 mm

Commit message: Hi
Parts:
- moved POTENTIOMETER 4.47 mm to (74.8, 38.5)
- moved LED-3 3.00 mm to (27.5, 50.5)
- moved LED-5 3.00 mm to (79.0, 50.5)
- moved ULTRASONICSENSOR 2.00 mm to (56.5, 48.0)
- moved U$1 2.00 mm to (50.5, 32.5)
- moved IRSENSOR1 1.00 mm to (73.0, 45.0)
- moved IRSENSOR2 1.00 mm to (41.0, 45.0)
- moved LDR1 1.00 mm to (93.0, 45.0)
- moved LDR2 1.00 mm to (21.0, 45.0)
- moved LED-2 1.00 mm to (6.00, 24.0)
- moved LED-6 1.00 mm to (100.0, 24.0)

Commit message: Most recent
Parts:
- moved PUSHBUTTON_RESISTOR 13.6 mm to (21.0, 35.0), turned to 135 degrees
- moved DIGITAL_PUSHBUTTON 7.21 mm to (16.0, 30.0), turned to 315 degrees
- moved SPEAKER 5.39 mm to (34.0, 29.0)
- moved BATTERY_CONNECTOR 2.24 mm to (29.4, 16.6)
Other:
- outline, holes or cut-outs redrawn

Commit message: component placement 95%
Parts:
- removed BATTERY_CONNECTOR: (no value), SparkFun-Connectors:MOLEX-1X3
- added BAT: (no value), SparkFun-Connectors:MOLEX-1X3
- moved SPEAKER 2.00 mm to (34.0, 31.0)
- renumbered DIGITAL_PUSHBUTTON to BUTTON, IRSENSOR1 to SENSOR2, IRSENSOR2 to SENSOR3, LDR1 to SENSOR1, LDR2 to SENSOR4, LED-2 to LED1, LED-3 to LED2, LED-5 to LED3, LED-6 to LED4, POTENTIOMETER to VR1, PUSHBUTTON_RESISTOR to R2, TOUCH_SENSOR_RESISTOR to R1, ULTRASONICSENSOR to ULTRA
Connections:
- net CAP_TOUCH_SEND_PIN renamed TOUCH
- net IR_SENSOR1_AO renamed SENSOR2
- net IR_SENSOR2_AO renamed SENSOR3
- net LDR1_AO renamed SENSOR1
- net LDR2_AO renamed SENSOR4
- removed net GND: LED1.3-GND, LED2.3-GND, LED3.3-GND, LED4.3-GND, R2.P$2, S1.NO1, SENSOR1.2, SENSOR2.2, SENSOR3.2, SENSOR4.2, SERVO1.1, SERVO2.1, SPEAKER.1, U$1.GND, U$1.GND1, ULTRA.4, VR1.1
- removed net SERVOVCC: SERVO1.2, SERVO2.2
- new net GND-ISO: LED1.3-GND, LED2.3-GND, LED3.3-GND, LED4.3-GND, R2.P$2, SENSOR1.2, SENSOR2.2, SENSOR3.2, SENSOR4.2, SERVO1.1, SERVO2.1, SPEAKER.1, U$1.GND1, ULTRA.4, VR1.1
- new net LEDS: U$1.D9
- new net N$6: SERVO1.3, U$1.D11
- new net N.C.: S1.NO1, U$1.GND
- net LED-1: no longer U$1.D9
- net N$9: now also BAT.3; no longer BATTERY_CONNECTOR.3
- net RAWIN: now also BAT.1; no longer BATTERY_CONNECTOR.1
- net VCC: now also BUTTON.3, SERVO1.2, SERVO2.2; no longer SERVO1.3, U$1.D11
Routing:
- added copper zone on layer 16, net N.C.
- removed copper zone on layer 16, net GND

Commit message: changes to physical
Parts:
- BAT: value (none) -> BAT
- S1: value (none) -> POWER
- moved LED1 37.6 mm to (39.0, 6.00)
- moved LED4 37.6 mm to (67.0, 6.00)
- moved SERVO2 29.0 mm to (18.0, 22.8), turned to 315 degrees
- moved SERVO1 24.1 mm to (85.0, 18.8), turned to 45 degrees
- moved BAT 8.06 mm to (40.4, 14.6), turned to 133.5 degrees
- moved VR1 6.08 mm to (73.8, 32.5), turned to 270 degrees
- moved R1 2.01 mm to (66.4, 29.5)
- moved BUTTON 2.00 mm to (14.0, 30.0)
- moved SPEAKER 2.00 mm to (34.0, 33.0)
- moved S1 1.41 mm to (71.0, 14.0)
Other:
- board text added: "BAT"
