File: pcb/v0.2/ArduinoNano LearningBot 4-21-18.brd (EAGLE design)
At the start: 106.9 x 55.1 mm, 19 parts

Commit message: almost there!
Parts:
- moved SERVO1 4.47 mm to (69.0, 6.77), turned to 135 degrees
- moved SERVO2 4.47 mm to (37.0, 6.77), turned to 45 degrees
- moved BUTTON 2.83 mm to (14.0, 32.0)
- moved R2 2.83 mm to (19.0, 37.0)
Connections:
- removed net GND-ISO: LED1.3-GND, LED2.3-GND, LED3.3-GND, LED4.3-GND, R2.P$2, SENSOR1.2, SENSOR2.2, SENSOR3.2, SENSOR4.2, SERVO1.1, SERVO2.1, SPEAKER.1, U$1.GND1, ULTRA.4, VR1.1
- removed net N.C.: S1.NO1, U$1.GND
- new net GND: LED1.3-GND, LED2.3-GND, LED3.3-GND, LED4.3-GND, R2.P$2, S1.NO1, SENSOR1.2, SENSOR2.2, SENSOR3.2, SENSOR4.2, SERVO1.1, SERVO2.1, SPEAKER.1, U$1.GND, U$1.GND1, ULTRA.4, VR1.1
Routing:
- added copper zone on layer 16, net GND
- removed copper zone on layer 16, net N.C.
Other:
- board text added: "+"
- board text added: "LearningBot v0.2 23/4/18 Nick & Rudi"

Commit message: Howdy
Parts:
- added U$2: TOUCHSENSOR, CapTouch:TOUCH1
- moved R1 3.70 mm to (69.0, 25.7), turned to 180 degrees
Connections:
- removed net LED-1: LED1.4-DIN
- net LEDS: now also LED1.4-DIN
- net TOUCH: now also U$2.P$1
Routing:
- net N$9: track 0.00 -> 57.4 mm
- net LDR1_DO: track 0.00 -> 55.1 mm
- net N$4: track 0.00 -> 51.6 mm
- net N$5: track 0.00 -> 51.5 mm
- net SENSOR2: track 0.00 -> 51.5 mm, vias 0 -> 2
- net RAWIN: track 0.00 -> 46.8 mm
- net SENSOR1: track 0.00 -> 46.0 mm
- net BUTTON: track 0.00 -> 43.5 mm, vias 0 -> 1
- net LEDS: track 0.00 -> 42.1 mm
- net TOUCH: track 0.00 -> 41.2 mm, vias 0 -> 1
- net SENSOR4: track 0.00 -> 38.3 mm
- net POTPIN: track 0.00 -> 30.4 mm
- net IR_SENSOR2_DO: track 0.00 -> 28.6 mm
- net GND: track 0.00 -> 28.0 mm, vias 0 -> 2
- net N$6: track 0.00 -> 27.7 mm
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