File: pcb/v0.3.514/ArduinoNano LearningBot 5-14-18.brd (EAGLE design)
At the start: 106.9 x 55.1 mm, 20 parts

Commit message: Hopefully, the last one
Parts:
- moved R1 6.99 mm to (64.5, 31.1), turned to 270 degrees
- moved SERVO2 4.94 mm to (40.7, 3.44), turned to 135 degrees
- moved S1 1.62 mm to (71.0, 13.7)
- moved ULTRA 0.32 mm to (56.5, 47.7)
- moved SERVO1 0.25 mm to (69.1, 7.00), turned to 225 degrees
- turned SPEAKER to 270 degrees
- renumbered U$2 to TOUCH
Connections:
- net N$6 renamed SERVO1
- net SERVO2_PIN renamed SERVO2
- removed net N$2: LED3.4-DIN
- removed net N$9: BAT.3, S1.C1
- new net VIN: BAT.1, S1.C1
- net GND: now also BAT.3; no longer S1.NO1
- net N$1: now also LED3.4-DIN
- net RAWIN: now also S1.NO1; no longer BAT.1
- net VCC: no longer BUTTON.3
Routing:
- net N$1: track 0.00 -> 64.3 mm, vias 0 -> 2
- net IR_SENSOR1_DO: track 0.00 -> 58.6 mm, vias 0 -> 2
- net N$9: track 57.4 -> 0.00 mm
- net VIN: track 0.00 -> 56.3 mm
- net SENSOR3: track 0.00 -> 52.3 mm, vias 0 -> 1
- net GND: track 28.0 -> 76.1 mm, vias 2 -> 5
- net LDR2_DO: track 0.00 -> 45.7 mm, vias 0 -> 2
- net TRIG_PIN: track 0.00 -> 37.5 mm, vias 0 -> 1
- net SENSOR4: track 38.3 -> 74.6 mm, vias 0 -> 3
- net ECHO_PIN: track 0.00 -> 32.5 mm, vias 0 -> 1
- net VCC: track 0.00 -> 31.7 mm
- net RAWIN: track 46.8 -> 31.9 mm, vias 0 -> 2
- net SENSOR2: track 51.5 -> 39.2 mm, vias 2 -> 1
- net SENSOR1: track 46.0 -> 53.6 mm, vias 0 -> 1
- net N$5: track 51.5 -> 58.8 mm
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Other:
- board text added: "BLACK"
- board text added: "D"
- board text added: "E"
- board text added: "G"
- board text added: "LearningBot v0.2.18427 KodingKreators Designed by Nick"
- board text added: "PWR SWITCH"
- board text added: "RED"
- board text added: "S"
- board text added: "T"
- board text added: "USB"
- board text added: "V"
- board text added: "YELLOW"
- board text removed: "LearningBot v0.2 23/4/18 Nick & Rudi"
